Commit message: Add cloned package files as regular folder

File: src/my_control/models/my_stair_robot/robot.urdf.xacro (robot description, xacro)
@@ -3,3 +3,4 @@
     <xacro:include filename="robot_core.xacro" />
     <xacro:include filename="robot_control.xacro" />
+    <xacro:include filename="robot_realsensed435i.xacro" />
 </robot>

File: src/my_control/models/my_stair_robot/robot_control.xacro (robot description, xacro)
@@ -17,5 +17,5 @@
             <publish_wheel_tf>true</publish_wheel_tf>
             <odometry_frame>odom</odometry_frame>
-            <robot_base_frame>chassis_link</robot_base_frame>
+            <robot_base_frame>base_link</robot_base_frame>
         </plugin>
     </gazebo>

File: src/my_control/models/my_stair_robot/robot_core.xacro (robot description, xacro)
@@ -14,4 +14,10 @@
     <material name="black"> <color rgba="0 0 0 1"/> </material>
     <material name="red"> <color rgba="1 0 0 1"/> </material>
+    <link name="base_link"></link>
+    <joint name="chassis_joint" type="fixed">
+            <parent link="base_link"/>
+            <child link="chassis_link"/>
+            <origin xyz="0 0 ${wheel_radius}"/>
+    </joint>
     <link name="chassis_link">
         <visual>
@@ -99,36 +105,3 @@
     </joint>
     <gazebo reference="wheel_castor_back_link"> <material>Gazebo/Red</material> </gazebo>
-    <!-- <joint name="camera_joint" type="fixed">
-        <parent link="chassis_link"/>
-        <child link="camera_link"/>
-        <origin xyz="0.1 0 0.2" rpy="0 0 0"/> </joint>
-    <gazebo reference="camera_link">
-        <sensor name="cameradepth" type="depth">
-            <camera name="camera">
-            <horizontal_fov>1.50098</horizontal_fov>
-            <image>
-                <width>640</width>
-                <height>480</height>
-                <format>R8G8B8</format>
-            </image>
-            <clip>
-                <near>0.1</near>
-                <far>100</far>
-            </clip>
-            </camera>
-            <always_on>1</always_on>
-            <update_rate>30</update_rate>
-            <visualize>true</visualize>
-            <plugin name="camera_controller" filename="libgazebo_ros_camera.so">
-            <ros>
-                <namespace>camera</namespace>
-                <remapping>custom_camera/image_raw:=color/image_raw</remapping>
-                <remapping>custom_camera/depth/image_raw:=depth/image_raw</remapping>
-            </ros>
-            <camera_name>camera</camera_name>
-            <frame_name>camera_depth_optical_frame</frame_name>
-            <hack_baseline>0.07</hack_baseline>
-            </plugin>
-        </sensor>
-        </gazebo> -->
 </robot>
