Commit message: add check_localize not yet

File: src/my_control/my_stair_robot/robot_core.xacro (robot description, xacro)
@@ -287,5 +287,5 @@
         <parent link="platform"/>
         <child link="camera_link"/>
-        <origin xyz="0.05 -0.43 0" rpy="1.5708 0 0"/>
+        <origin xyz="0.04 -0.0 0" rpy="1.5708 0 0"/>
     </joint>
     <link name="camera_link">
@@ -297,3 +297,16 @@
         </visual>
     </link>
+    <joint name="imubody_joint" type="fixed">
+        <parent link="base_link"/>
+        <child link="imubody_link"/>
+        <origin xyz="-0.4 -0.2 0.0" rpy="0 0 0"/>
+    </joint>
+    <link name="imubody_link">
+        <visual>
+            <geometry>
+                <box size="0.01 0.03 0.01"/>
+            </geometry>
+            <material name="black"/>
+        </visual>
+    </link>
 </robot>

Commit message: 

File: src/my_control/my_stair_robot/robot_core.xacro (robot description, xacro)
@@ -1,4 +1,18 @@
 <?xml version="1.0"?>
 <robot xmlns:xacro="http://www.ros.org/wiki/xacro" name="my_stair_robot">
+  <material name="red">
+    <color rgba="1.0 0.0 0.0 1.0"/>
+  </material>
+  <material name="black">
+    <color rgba="0.0 0.0 0.0 1.0"/>
+  </material>
+  <material name="gray_blue">
+    <color rgba="0.792 0.819 0.933 1.0"/>
+  </material>
+  <link name="base_footprint"/>
+  <joint name="base_footprint_joint" type="fixed">
+    <parent link="base_footprint"/>
+    <child link="base_link"/>
+    <origin xyz="0 0 0.05" rpy="0 0 0"/> </joint>
   <link name="base_link">
     <inertial>
@@ -12,5 +26,5 @@
         <mesh filename="package://my_control/my_stair_robot/meshes/base_link.STL" />
       </geometry>
-      <material name=""><color rgba="0.792156862745098 0.819607843137255 0.933333333333333 1" /></material>
+      <material name="gray_blue"/>
     </visual>
     <collision>
@@ -29,14 +43,10 @@
     <visual>
       <origin xyz="0 0 0" rpy="0 0 0" />
-      <geometry>
-        <mesh filename="package://my_control/my_stair_robot/meshes/left_wheel.STL" />
-      </geometry>
-      <material name=""><color rgba="0.796078431372549 0.823529411764706 0.937254901960784 1" /></material>
-    </visual>
-    <collision>
-      <origin xyz="0 0 0" rpy="0 0 0" />
-      <geometry>
-        <mesh filename="package://my_control/my_stair_robot/meshes/left_wheel.STL" />
-      </geometry>
+      <geometry><mesh filename="package://my_control/my_stair_robot/meshes/left_wheel.STL" /></geometry>
+      <material name="gray_blue"/>
+    </visual>
+    <collision>
+      <origin xyz="0 0 0" rpy="0 0 0" />
+      <geometry><mesh filename="package://my_control/my_stair_robot/meshes/left_wheel.STL" /></geometry>
     </collision>
   </link>
@@ -57,14 +67,10 @@
     <visual>
       <origin xyz="0 0 0" rpy="0 0 0" />
-      <geometry>
-        <mesh filename="package://my_control/my_stair_robot/meshes/right_wheel.STL" />
-      </geometry>
-      <material name=""><color rgba="0.796078431372549 0.823529411764706 0.937254901960784 1" /></material>
-    </visual>
-    <collision>
-      <origin xyz="0 0 0" rpy="0 0 0" />
-      <geometry>
-        <mesh filename="package://my_control/my_stair_robot/meshes/right_wheel.STL" />
-      </geometry>
+      <geometry><mesh filename="package://my_control/my_stair_robot/meshes/right_wheel.STL" /></geometry>
+      <material name="gray_blue"/>
+    </visual>
+    <collision>
+      <origin xyz="0 0 0" rpy="0 0 0" />
+      <geometry><mesh filename="package://my_control/my_stair_robot/meshes/right_wheel.STL" /></geometry>
     </collision>
   </link>
@@ -86,5 +92,5 @@
       <origin xyz="0 0 0" rpy="0 0 0" />
       <geometry><mesh filename="package://my_control/my_stair_robot/meshes/rear_caster.STL" /></geometry>
-      <material name=""><color rgba="0.792156862745098 0.819607843137255 0.933333333333333 1" /></material>
+      <material name="gray_blue"/>
     </visual>
     <collision>
@@ -98,5 +104,4 @@
     <child link="rear_caster" />
     <axis xyz="0 0 1" />
-    <dynamics damping="0.1" friction="0.02" />
   </joint>
   <link name="rear_caster_wheel">
@@ -109,5 +114,5 @@
       <origin xyz="0 0 0" rpy="0 0 0" />
       <geometry><mesh filename="package://my_control/my_stair_robot/meshes/rear_caster_wheel.STL" /></geometry>
-      <material name=""><color rgba="0.792156862745098 0.819607843137255 0.933333333333333 1" /></material>
+      <material name="gray_blue"/>
     </visual>
     <collision>
@@ -121,5 +126,4 @@
     <child link="rear_caster_wheel" />
     <axis xyz="-0.00665576114394258 0 -0.99997785017649" />
-    <dynamics damping="0.1" friction="0.02" />
   </joint>
   <link name="front_left_arm">
@@ -132,5 +136,5 @@
       <origin xyz="0 0 0" rpy="0 0 0" />
       <geometry><mesh filename="package://my_control/my_stair_robot/meshes/front_left_arm.STL" /></geometry>
-      <material name=""><color rgba="0.792156862745098 0.819607843137255 0.933333333333333 1" /></material>
+      <material name="gray_blue"/>
     </visual>
     <collision>
@@ -144,6 +148,4 @@
     <child link="front_left_arm" />
     <axis xyz="0 0 1" />
-    <limit effort="236" velocity="2.6" />
-    <dynamics damping="0.1" friction="0.02" />
   </joint>
   <link name="left_arm_f">
@@ -156,5 +158,5 @@
       <origin xyz="0 0 0" rpy="0 0 0" />
       <geometry><mesh filename="package://my_control/my_stair_robot/meshes/left_arm_f.STL" /></geometry>
-      <material name=""><color rgba="0.792156862745098 0.819607843137255 0.933333333333333 1" /></material>
+      <material name="gray_blue"/>
     </visual>
     <collision>
@@ -179,5 +181,5 @@
       <origin xyz="0 0 0" rpy="0 0 0" />
       <geometry><mesh filename="package://my_control/my_stair_robot/meshes/front_right_arm.STL" /></geometry>
-      <material name=""><color rgba="0.792156862745098 0.819607843137255 0.933333333333333 1" /></material>
+      <material name="gray_blue"/>
     </visual>
     <collision>
@@ -191,6 +193,4 @@
     <child link="front_right_arm" />
     <axis xyz="0 0 1" />
-    <limit effort="236" velocity="2.6" />
-    <dynamics damping="0.1" friction="0.02" />
   </joint>
   <link name="right_arm_f">
@@ -203,5 +203,5 @@
       <origin xyz="0 0 0" rpy="0 0 0" />
       <geometry><mesh filename="package://my_control/my_stair_robot/meshes/right_arm_f.STL" /></geometry>
-      <material name=""><color rgba="0.792156862745098 0.819607843137255 0.933333333333333 1" /></material>
+      <material name="gray_blue"/>
     </visual>
     <collision>
@@ -226,9 +226,6 @@
       <origin xyz="0 0 0" rpy="0 0 0" />
       <geometry><mesh filename="package://my_control/my_stair_robot/meshes/rear_left_arm.STL" /></geometry>
-    </visual>
-    <collision>
-      <origin xyz="0 0 0" rpy="0 0 0" />
-      <geometry><mesh filename="package://my_control/my_stair_robot/meshes/rear_left_arm.STL" /></geometry>
-    </collision>
+      <material name="gray_blue"/>
+    </visual>
   </link>
   <joint name="rearleftarm" type="continuous">
@@ -248,9 +245,6 @@
       <origin xyz="0 0 0" rpy="0 0 0" />
       <geometry><mesh filename="package://my_control/my_stair_robot/meshes/rear_right_arm.STL" /></geometry>
-    </visual>
-    <collision>
-      <origin xyz="0 0 0" rpy="0 0 0" />
-      <geometry><mesh filename="package://my_control/my_stair_robot/meshes/rear_right_arm.STL" /></geometry>
-    </collision>
+      <material name="gray_blue"/>
+    </visual>
   </link>
   <joint name="rearrightarm" type="continuous">
@@ -270,4 +264,5 @@
       <origin xyz="0 0 0" rpy="0 0 0" />
       <geometry><mesh filename="package://my_control/my_stair_robot/meshes/platform.STL" /></geometry>
+      <material name="gray_blue"/>
     </visual>
     <collision>
@@ -284,29 +279,25 @@
     <dynamics damping="0.1" friction="0.02" />
   </joint>
-    <joint name="camera_joint" type="fixed">
-        <parent link="platform"/>
-        <child link="camera_link"/>
-        <origin xyz="0.04 -0.0 0" rpy="1.5708 0 0"/>
-    </joint>
-    <link name="camera_link">
-        <visual>
-            <geometry>
-                <box size="0.020 0.06 0.03"/>
-            </geometry>
-            <material name="red"/>
-        </visual>
-    </link>
-    <joint name="imubody_joint" type="fixed">
-        <parent link="base_link"/>
-        <child link="imubody_link"/>
-        <origin xyz="-0.4 -0.2 0.0" rpy="0 0 0"/>
-    </joint>
-    <link name="imubody_link">
-        <visual>
-            <geometry>
-                <box size="0.01 0.03 0.01"/>
-            </geometry>
-            <material name="black"/>
-        </visual>
-    </link>
+  <joint name="camera_joint" type="fixed">
+    <parent link="platform"/>
+    <child link="camera_link"/>
+    <origin xyz="0.04 -0.0 0" rpy="1.5708 0 0"/>
+  </joint>
+  <link name="camera_link">
+    <visual>
+      <geometry><box size="0.020 0.06 0.03"/></geometry>
+      <material name="red"/>
+    </visual>
+  </link>
+  <joint name="imubody_joint" type="fixed">
+    <parent link="base_link"/>
+    <child link="imubody_link"/>
+    <origin xyz="-0.4 -0.2 0.0" rpy="0 0 0"/>
+  </joint>
+  <link name="imubody_link">
+    <visual>
+      <geometry><box size="0.01 0.03 0.01"/></geometry>
+      <material name="black"/>
+    </visual>
+  </link>
 </robot>
